Commit message: Add battery to turtlebot

File: rl_passage_formation/data/turtlebot3.urdf (robot description, URDF)
Before this commit: robot turtlebot3_burger, 7 links, 6 joints
Links:
- added link base_battery, mass 0.13; collision box size=0.12 0.03 0.02; visual box size=0.12 0.03 0.02
- added link base_cam, mass 0.01
Joints:
- added joint battery_joint: type fixed, parent base_link, child base_battery, origin xyz=0.0 0 0.02 rpy=0 0 0
- added joint camera_joint: type fixed, parent base_link, child base_cam, origin xyz=0.01 0.0 0.11 rpy=0 0 0
